File: Board/CT2960_Riser/CT2960_Riser.sch (KiCad schematic (older format))
At the start: 64 parts, among them IC1 74LVC8T245, IC2 74LVC8T245, IC3 74LVC8T245, IC4 74LVC8T245, IC5 74LVC8T245, IC6 74LVC8T245, J1 Conn_02x20_Odd_Even, J2 Conn_02x12_Top_Bottom, J3 Bus_ISA_16bit, J4 Conn_02x20_Odd_Even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

Commit message: Commit 06052019
Connections:
- net IOR: now also D4.2 (A)
- net IOW: now also D3.2 (A)
- net at IC2.4 (A2), J1.22 (Pin_22), U1.1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: no longer D3.2 (A)
- net at IC2.5 (A3), J1.24 (Pin_24), U1.2: no longer D4.2 (A)
Other:
- moved on the sheet: C11, C12, C21, C22, D3, D4, R12, R9
